Commit message: Fix the joint limits divergence

File: pai_bringup/config/control/so_arm101.ros2_control.xacro (robot description, xacro)
@@ -1,7 +1,24 @@
 <?xml version="1.0" ?>
 <robot xmlns:xacro="http://www.ros.org/wiki/xacro">
+  <!-- Shared ros2_control definition for all hardware backends.
+       MuJoCo, Gazebo, real hardware, and mock_components all use this macro
+       so that joint IDs, gains, and offsets are defined in exactly one place.
+       MuJoCo-specific params (mujoco_model, sim_speed_factor, camera_*) are
+       only used when ros2_control_hardware_type == 'mujoco'.  Camera sensors
+       are added when camera_frame is non-empty. -->
   <xacro:macro
     name="ros2_control"
-    params="prefix ros2_control_hardware_type usb_port"
+    params="
+      prefix
+      ros2_control_hardware_type
+      usb_port:=''
+      mujoco_model:=''
+      sim_speed_factor:='1.0'
+      camera_publish_rate:='10.0'
+      camera_frame:=''
+      camera_info_topic:='/camera/info'
+      camera_image_topic:='/camera'
+      camera_depth_topic:='/camera/depth'
+    "
   >
     <ros2_control name="SO_ARM101" type="system">
@@ -16,7 +33,7 @@
         <xacro:if value="${ros2_control_hardware_type == 'mujoco'}">
           <plugin>mujoco_ros2_control/MujocoSystemInterface</plugin>
-          <param name="mujoco_model">
-            $(find so_arm101_description)/mjcf/scene.xml
-          </param>
+          <param name="mujoco_model">${mujoco_model}</param>
+          <param name="sim_speed_factor">${sim_speed_factor}</param>
+          <param name="camera_publish_rate">${camera_publish_rate}</param>
         </xacro:if>
         <xacro:if value="${ros2_control_hardware_type == 'gazebo'}">
@@ -27,5 +44,8 @@
         <param name="initial_position">0.0</param>
         <param name="id">1</param>
-        <param name="p_cofficient">8</param>
+        <!-- Lower P gain (8 vs 16) for the base joint to reduce oscillation
+             under the higher inertia of the full arm above it.
+             Note: param name matches feetech_ros2_driver's expected spelling. -->
+        <param name="p_coefficient">8</param>
         <param name="offset">2048</param>
         <command_interface name="position">
@@ -40,9 +60,8 @@
       <joint name="${prefix}shoulder_lift_joint">
         <param name="id">2</param>
-        <param name="p_cofficient">16</param>
+        <param name="p_coefficient">16</param>
         <param name="offset">2048</param>
         <param name="initial_position">0.0</param>
         <command_interface name="position">
-          <!-- PID gains: only read by gz_ros2_control (Gazebo hardware interface) -->
           <param name="p">100.0</param>
           <param name="i">0.1</param>
@@ -55,8 +74,7 @@
         <param name="id">3</param>
         <param name="offset">2048</param>
-        <param name="p_cofficient">16</param>
+        <param name="p_coefficient">16</param>
         <param name="initial_position">0.0</param>
         <command_interface name="position">
-          <!-- PID gains: only read by gz_ros2_control (Gazebo hardware interface) -->
           <param name="p">100.0</param>
           <param name="i">0.1</param>
@@ -69,8 +87,7 @@
         <param name="id">4</param>
         <param name="offset">2048</param>
-        <param name="p_cofficient">16</param>
+        <param name="p_coefficient">16</param>
         <param name="initial_position">0.0</param>
         <command_interface name="position">
-          <!-- PID gains: only read by gz_ros2_control (Gazebo hardware interface) -->
           <param name="p">100.0</param>
           <param name="i">0.1</param>
@@ -83,8 +100,7 @@
         <param name="id">5</param>
         <param name="offset">2048</param>
-        <param name="p_cofficient">16</param>
+        <param name="p_coefficient">16</param>
         <param name="initial_position">0.0</param>
         <command_interface name="position">
-          <!-- PID gains: only read by gz_ros2_control (Gazebo hardware interface) -->
           <param name="p">100.0</param>
           <param name="i">0.1</param>
@@ -97,8 +113,7 @@
         <param name="id">6</param>
         <param name="offset">2048</param>
-        <param name="p_cofficient">16</param>
+        <param name="p_coefficient">16</param>
         <param name="initial_position">0.0</param>
         <command_interface name="position">
-          <!-- PID gains: only read by gz_ros2_control (Gazebo hardware interface) -->
           <param name="p">100.0</param>
           <param name="i">0.1</param>
@@ -108,4 +123,13 @@
         <state_interface name="velocity" />
       </joint>
+      <!-- Camera sensor: only added when camera_frame is provided (MuJoCo sim) -->
+      <xacro:if value="${camera_frame != ''}">
+        <sensor name="camera">
+          <param name="frame_name">${camera_frame}</param>
+          <param name="info_topic">${camera_info_topic}</param>
+          <param name="image_topic">${camera_image_topic}</param>
+          <param name="depth_topic">${camera_depth_topic}</param>
+        </sensor>
+      </xacro:if>
     </ros2_control>
   </xacro:macro>

File: pai_bringup/mjcf/so_arm101.xml.xacro (robot description, xacro)
@@ -110,5 +110,5 @@
           name="shoulder_pan_joint"
           type="hinge"
-          range="-1.9198621771937616 1.9198621771937634"
+          range="-1.91986 1.91986"
           class="sts3215"
         />
@@ -170,5 +170,5 @@
             name="shoulder_lift_joint"
             type="hinge"
-            range="-1.7453292519943224 1.7453292519943366"
+            range="-1.74533 1.74533"
             class="sts3215"
           />
@@ -216,5 +216,5 @@
               name="elbow_flex_joint"
               type="hinge"
-              range="-1.69 1.69"
+              range="-1.69 1.54"
               class="sts3215"
             />
@@ -276,5 +276,5 @@
                 name="wrist_flex_joint"
                 type="hinge"
-                range="-1.6580628494556928 1.6580627293335335"
+                range="-1.6 1.6"
                 class="sts3215"
               />
@@ -322,5 +322,5 @@
                   name="wrist_roll_joint"
                   type="hinge"
-                  range="-2.7438472969992493 2.841206309382605"
+                  range="-2.3 2.3"
                   class="sts3215"
                 />
@@ -374,5 +374,5 @@
                     name="gripper_joint"
                     type="hinge"
-                    range="-0.17453297762778586 1.7453291995659765"
+                    range="0.0 1.0"
                     class="sts3215"
                   />
@@ -427,5 +427,5 @@
       joint="elbow_flex_joint"
       forcerange="-3.35 3.35"
-      ctrlrange="-1.69 1.69"
+      ctrlrange="-1.69 1.54"
     />
     <position
@@ -434,5 +434,5 @@
       joint="wrist_flex_joint"
       forcerange="-3.35 3.35"
-      ctrlrange="-1.65806 1.65806"
+      ctrlrange="-1.6 1.6"
     />
     <position
@@ -441,5 +441,5 @@
       joint="wrist_roll_joint"
       forcerange="-3.35 3.35"
-      ctrlrange="-2.74385 2.84121"
+      ctrlrange="-2.3 2.3"
     />
     <position
@@ -448,5 +448,5 @@
       joint="gripper_joint"
       forcerange="-3.35 3.35"
-      ctrlrange="-0.17453 1.74533"
+      ctrlrange="0.0 1.0"
     />
   </actuator>

File: pai_bringup/urdf/so_arm101_mujoco.urdf.xacro (robot description, xacro)
@@ -22,73 +22,13 @@
     <origin xyz="0.0 0.0 0.5" rpy="0 2.356 0.0"/>
   </joint>
-  <!-- ros2_control information including camera sensor -->
-  <ros2_control name="MujocoSystem" type="system">
-    <hardware>
-      <plugin>mujoco_ros2_control/MujocoSystemInterface</plugin>
-      <param name="mujoco_model">$(arg mujoco_model)</param>
-      <param name="sim_speed_factor">1.0</param>
-      <param name="camera_publish_rate">10.0</param>
-    </hardware>
-    <joint name="$(arg prefix)shoulder_pan_joint">
-      <param name="initial_position">0.0</param>
-      <param name="id">1</param>
-      <param name="p_cofficient">8</param>
-      <param name="offset">2048</param>
-      <command_interface name="position" />
-      <state_interface name="position" />
-      <state_interface name="velocity" />
-    </joint>
-    <joint name="$(arg prefix)shoulder_lift_joint">
-      <param name="id">2</param>
-      <param name="p_cofficient">16</param>
-      <param name="offset">2125</param>
-      <param name="initial_position">0.0</param>
-      <command_interface name="position" />
-      <state_interface name="position" />
-      <state_interface name="velocity" />
-    </joint>
-    <joint name="$(arg prefix)elbow_flex_joint">
-      <param name="id">3</param>
-      <param name="offset">2080</param>
-      <param name="p_cofficient">16</param>
-      <param name="initial_position">0.0</param>
-      <command_interface name="position" />
-      <state_interface name="position" />
-      <state_interface name="velocity" />
-    </joint>
-    <joint name="$(arg prefix)wrist_flex_joint">
-      <param name="id">4</param>
-      <param name="offset">3110</param>
-      <param name="p_cofficient">16</param>
-      <param name="initial_position">0.0</param>
-      <command_interface name="position" />
-      <state_interface name="position" />
-      <state_interface name="velocity" />
-    </joint>
-    <joint name="$(arg prefix)wrist_roll_joint">
-      <param name="id">5</param>
-      <param name="offset">1024</param>
-      <param name="p_cofficient">16</param>
-      <param name="initial_position">0.0</param>
-      <command_interface name="position" />
-      <state_interface name="position" />
-      <state_interface name="velocity" />
-    </joint>
-    <joint name="$(arg prefix)gripper_joint">
-      <param name="id">6</param>
-      <param name="offset">2070</param>
-      <param name="p_cofficient">16</param>
-      <param name="initial_position">0.0</param>
-      <command_interface name="position" />
-      <state_interface name="position" />
-      <state_interface name="velocity" />
-    </joint>
-    <!-- Camera informatiom -->
-    <sensor name="camera">
-      <param name="frame_name">camera_color_mujoco_frame</param>
-      <param name="info_topic">/camera/info</param>
-      <param name="image_topic">/camera</param>
-      <param name="depth_topic">/camera/depth</param>
-    </sensor>
-  </ros2_control>
+  <!-- ros2_control: uses the shared macro (single definition for all backends).
+       Joint IDs, gains, and offsets are defined once in so_arm101.ros2_control.xacro.
+       Camera sensor is enabled by passing camera_frame. -->
+  <xacro:include filename="$(find pai_bringup)/config/control/so_arm101.ros2_control.xacro" />
+  <xacro:ros2_control
+    prefix="$(arg prefix)"
+    ros2_control_hardware_type="mujoco"
+    mujoco_model="$(arg mujoco_model)"
+    camera_frame="camera_color_mujoco_frame"
+  />
 </robot>
