Commit message: Add support for wrist and static cameras in real and simulation.
Signed-off-by: Franco Cipollone <franco.c@ekumenlabs.com>

File: pai_bringup/mjcf/so_arm101.xml.xacro (robot description, xacro)
@@ -397,4 +397,8 @@
                   />
                 </body>
+                <!-- Wrist camera: MuJoCo cameras use OpenGL convention (-Z forward, +Y up).
+                     euler derived from URDF optical RPY (2.618 0 0) via R_mj = R_urdf * Rx(π). -->
+                <camera name="wrist_camera" fovy="55" mode="fixed" resolution="640 480"
+                        pos="0.0 0.065 -0.03" euler="-0.5236 0 0"/>
               </body>
             </body>
@@ -402,7 +406,8 @@
         </body>
       </body>
-      <!-- Camera: elevated above workspace for full scene visibility (table, tray, cubes, gripper) -->
-      <site name="camera_color_mujoco_frame" pos="0.25 0.0 0.55" euler="0 -0.7 0"/>
-      <camera name="camera" fovy="52" mode="fixed" resolution="1280 720" pos="0.25 0.0 0.55" euler="0 -0.7 0"/>
+      <!-- Static camera: elevated above base_link, tilted 30° toward +X.
+           euler derived from URDF optical RPY (3.6652 0 -1.5708) via R_mj = R_urdf * Rx(π). -->
+      <camera name="static_camera" fovy="55" mode="fixed" resolution="640 480"
+              pos="0.0 0.0 0.50" euler="0 -0.5236 -1.5708"/>
     </body>
   </worldbody>

File: pai_bringup/urdf/so_arm101_mujoco.urdf.xacro (robot description, xacro)
@@ -15,12 +15,10 @@
     x="$(arg arm_base_x)" y="$(arg arm_base_y)" z="$(arg arm_base_z)"
     roll="$(arg arm_base_roll)" pitch="$(arg arm_base_pitch)" yaw="$(arg arm_base_yaw)" />
-  <!-- Overhead camera link -->
-  <link name="camera_color_mujoco_frame"/>
-  <joint name="camera_color_mujoco_joint" type="fixed">
-    <parent link="base_link"/>
-    <child link="camera_color_mujoco_frame"/>
-    <origin xyz="0.0 0.0 0.5" rpy="0 2.356 0.0"/>
-  </joint>
-  <!-- ros2_control information including camera sensor -->
+  <!-- Camera frames (wrist + static).
+       Poses are hardcoded here (not launch-configurable) because the MJCF
+       camera poses use MuJoCo/OpenGL convention and must stay in sync. -->
+  <xacro:include filename="$(find pai_bringup)/urdf/cameras.xacro" />
+  <xacro:pai_cameras prefix="$(arg prefix)" />
+  <!-- ros2_control information including camera sensors -->
   <ros2_control name="MujocoSystem" type="system">
     <hardware>
@@ -84,10 +82,17 @@
       <state_interface name="velocity" />
     </joint>
-    <!-- Camera informatiom -->
-    <sensor name="camera">
-      <param name="frame_name">camera_color_mujoco_frame</param>
-      <param name="info_topic">/camera/info</param>
-      <param name="image_topic">/camera</param>
-      <param name="depth_topic">/camera/depth</param>
+    <!-- Wrist camera (MuJoCo camera name must match sensor name) -->
+    <sensor name="wrist_camera">
+      <param name="frame_name">wrist_camera_link</param>
+      <param name="info_topic">/wrist_camera/camera_info</param>
+      <param name="image_topic">/wrist_camera/image_raw</param>
+      <param name="depth_topic">/wrist_camera/depth</param>
+    </sensor>
+    <!-- Static camera -->
+    <sensor name="static_camera">
+      <param name="frame_name">static_camera_link</param>
+      <param name="info_topic">/static_camera/camera_info</param>
+      <param name="image_topic">/static_camera/image_raw</param>
+      <param name="depth_topic">/static_camera/depth</param>
     </sensor>
   </ros2_control>

File: pai_bringup/urdf/so_arm_gz.urdf.xacro (robot description, xacro)
@@ -13,4 +13,7 @@
   <xacro:arg name="prefix" default="" />
   <xacro:arg name="color" default="0.2 0.7 0.85 1.0" />
+  <!-- Static camera pose – override at launch to match your physical setup -->
+  <xacro:arg name="cam_static_xyz" default="0.0 0.0 0.50" />
+  <xacro:arg name="cam_static_rpy" default="3.6652 0.0 -1.5708" />
   <!-- Pose arguments for robot positioning -->
   <xacro:arg name="x" default="0.0" />
@@ -33,4 +36,69 @@
                    pitch="$(arg pitch)"
                    yaw="$(arg yaw)" />
+  <!-- Camera frames (wrist + static).
+       include_inertia=true adds a minimal <inertial> to each camera link so
+       the URDF→SDF converter keeps them (links without inertia are dropped). -->
+  <xacro:include filename="$(find pai_bringup)/urdf/cameras.xacro" />
+  <xacro:pai_cameras prefix="$(arg prefix)"
+    cam_static_xyz="$(arg cam_static_xyz)"
+    cam_static_rpy="$(arg cam_static_rpy)"
+    include_inertia="true" />
+  <!-- Preserve camera fixed joints during URDF→SDF conversion -->
+  <gazebo reference="wrist_camera_joint">
+    <preserveFixedJoint>true</preserveFixedJoint>
+  </gazebo>
+  <gazebo reference="static_camera_joint">
+    <preserveFixedJoint>true</preserveFixedJoint>
+  </gazebo>
+  <!--
+    Gazebo camera sensors.
+    The camera links from cameras.xacro use the ROS optical convention
+    (Z-forward, X-right, Y-down).  Gazebo camera sensors look along +X
+    with +Z up, so we add a sensor <pose> rotation to compensate:
+      pitch=-π/2, yaw=+π/2  ⇒  sensor +X → link +Z (forward),
+                                 sensor +Z → link -Y (up).
+  -->
+  <gazebo reference="wrist_camera_link">
+    <sensor name="wrist_camera" type="camera">
+      <gz_frame_id>wrist_camera_link</gz_frame_id>
+      <pose>0 0 0 0 -1.5708 1.5708</pose>
+      <always_on>true</always_on>
+      <update_rate>30</update_rate>
+      <camera>
+        <horizontal_fov>1.2217</horizontal_fov>
+        <image>
+          <width>640</width>
+          <height>480</height>
+          <format>R8G8B8</format>
+        </image>
+        <clip>
+          <near>0.01</near>
+          <far>100</far>
+        </clip>
+      </camera>
+      <topic>wrist_camera/image_raw</topic>
+    </sensor>
+  </gazebo>
+  <gazebo reference="static_camera_link">
+    <sensor name="static_camera" type="camera">
+      <gz_frame_id>static_camera_link</gz_frame_id>
+      <pose>0 0 0 0 -1.5708 1.5708</pose>
+      <always_on>true</always_on>
+      <update_rate>30</update_rate>
+      <camera>
+        <horizontal_fov>1.2217</horizontal_fov>
+        <image>
+          <width>640</width>
+          <height>480</height>
+          <format>R8G8B8</format>
+        </image>
+        <clip>
+          <near>0.01</near>
+          <far>100</far>
+        </clip>
+      </camera>
+      <topic>static_camera/image_raw</topic>
+    </sensor>
+  </gazebo>
   <!-- parameters -->
   <xacro:arg name="simulation_controllers" default="" />

File: pai_bringup/urdf/so_arm_real.urdf.xacro (robot description, xacro)
@@ -15,4 +15,7 @@
   <xacro:arg name="prefix" default="" />
   <xacro:arg name="color" default="0.2 0.7 0.85 1.0" />
+  <!-- Static camera pose – override at launch to match your physical setup -->
+  <xacro:arg name="cam_static_xyz" default="0.0 0.0 0.50" />
+  <xacro:arg name="cam_static_rpy" default="3.6652 0.0 -1.5708" />
   <!-- World link (required as parent for the base fixed joint) -->
   <link name="world" />
@@ -20,4 +23,9 @@
   <xacro:include filename="$(arg urdf_file)" />
   <xacro:so_arm101 prefix="$(arg prefix)" color="$(arg color)" />
+  <!-- Camera frames (wrist + static) -->
+  <xacro:include filename="$(find pai_bringup)/urdf/cameras.xacro" />
+  <xacro:pai_cameras prefix="$(arg prefix)"
+    cam_static_xyz="$(arg cam_static_xyz)"
+    cam_static_rpy="$(arg cam_static_rpy)" />
   <!-- ros2_control description -->
   <xacro:include filename="$(arg ros2_control_file)" />
